Commit message: change_lidar_pos

File: robots/youbot_base_only.urdf.xacro (robot description, xacro)
@@ -27,5 +27,5 @@
   <!-- base laser front -->
   <xacro:hokuyo_urg04_laser name="base_laser_front" parent="base" ros_topic="scan_front" update_rate="10" min_angle="-1.57" max_angle="1.57">
-    <origin xyz="0.3 0 -0.03" rpy="0 0 0"/>
+    <origin xyz="0.3 0 0.08" rpy="0 0 0"/>
   </xacro:hokuyo_urg04_laser>
 </robot>
